Commit message: Lab 4 completed

File: src/my_r2d2/urdf/r2d2.xacro (robot description, xacro)
@@ -8,4 +8,5 @@
   <xacro:property name="wheeldiam" value="0.07" />
   <xacro:property name="pi" value="3.1415" />
+  <xacro:property name="legwidth" value="0.1" />
   <material name="blue">
     <color rgba="0 0 0.8 1"/>
@@ -42,5 +43,5 @@
         <origin xyz="0 0 0" rpy="${pi/2} 0 0" />
         <geometry>
-          <cylinder radius="${wheeldiam/2}" length="0.1"/>
+          <cylinder radius="${wheeldiam/2}" length="${legwidth}"/>
         </geometry>
         <material name="black"/>
@@ -49,5 +50,5 @@
         <origin xyz="0 0 0" rpy="${pi/2} 0 0" />
         <geometry>
-          <cylinder radius="${wheeldiam/2}" length="0.1"/>
+          <cylinder radius="${wheeldiam/2}" length="${legwidth}"/>
         </geometry>
       </collision>
@@ -65,5 +66,5 @@
       <visual>
         <geometry>
-          <box size="${leglen} 0.1 0.2"/>
+          <box size="${leglen} ${legwidth} 0.2"/>
         </geometry>
         <origin xyz="0 0 -${leglen/2}" rpy="0 ${pi/2} 0"/>
@@ -72,5 +73,5 @@
       <collision>
         <geometry>
-          <box size="${leglen} 0.1 0.2"/>
+          <box size="${leglen} ${legwidth} 0.2"/>
         </geometry>
         <origin xyz="0 0 -${leglen/2}" rpy="0 ${pi/2} 0"/>
@@ -86,5 +87,5 @@
       <visual>
         <geometry>
-          <box size="${baselen} 0.1 0.1"/>
+          <box size="${baselen} ${legwidth} ${legwidth}"/>
         </geometry>
         <material name="white"/>
@@ -92,5 +93,5 @@
       <collision>
         <geometry>
-          <box size="${baselen} 0.1 0.1"/>
+          <box size="${baselen} ${legwidth} ${legwidth}"/>
         </geometry>
       </collision>
@@ -234,3 +235,9 @@
     <origin xyz="${.707*width+0.04} 0 ${.707*width}"/>
   </joint>
+ <link name="base_footprint"/>
+ <joint name="base_to_footprint" type="fixed">
+    <child link="base_link"/>
+    <parent link = "base_footprint"/>
+    <origin xyz="0 0 ${bodylen/2 + legwidth + wheeldiam}"/>
+ </joint>
 </robot>

Commit message: Lab 5 complete

File: src/my_r2d2/urdf/r2d2.xacro (robot description, xacro)
@@ -241,3 +241,9 @@
     <origin xyz="0 0 ${bodylen/2 + legwidth + wheeldiam}"/>
  </joint>
+ <link name="eye"/>
+ <joint name="eye_to_lense" type="fixed">
+    <child link="eye"/>
+    <parent link="lens"/>
+    <origin xyz="0 0 0" rpy="${pi/2} -${pi} ${pi/2}"/>
+ </joint>
 </robot>
